File: EquipmentBox1/EquipmentBox1.kicad_pcb (KiCad board)
At the start: 2 copper layers, 272.5 x 41 mm, 11 parts, among them J1 UAC16-9, J10 UAV20-5, J11 UAC28-2, J2 UAC16-9, J3 UAC16-9, J4 UAC16-9, J5 UAC16-8, J6 UAC16-8, J7 UAC16-8, J8 UAC16-8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

Commit message: 已打样测试两版，第三版暂未修改
Parts:
- added J12: 430450612, Molex:430450612, B.Cu at (270.0, 59.5)
- added J13: 430452212, Molex:430452212, B.Cu at (316.0, 59.5)
- added J14: 430452412, Molex:430452412, B.Cu at (287.0, 59.5)
- added J15: XT60F, Connector_AMASS:AMASS_XT60-F_1x02_P7.20mm_Vertical, B.Cu at (185.6, 45.0)
- added J16: XT60F, Connector_AMASS:AMASS_XT60-F_1x02_P7.20mm_Vertical, B.Cu at (225.6, 45.0)
- added R1: 1K, Resistor_SMD:R_0402_1005Metric, F.Cu at (321.0, 44.0)
- added R2: 1K, Resistor_SMD:R_0402_1005Metric, F.Cu at (321.0, 47.0)
- added R3: 1K, Resistor_SMD:R_0402_1005Metric, F.Cu at (320.9, 50.0)
- added R4: 1K, Resistor_SMD:R_0402_1005Metric, F.Cu at (321.0, 53.0)
Connections:
- J1 pad 1: unconnected-(J1-Pin_1-Pad1) -> +5V
- J1 pad 2: unconnected-(J1-Pin_2-Pad2) -> /PWM3_Z-B
- J1 pad 3: unconnected-(J1-Pin_3-Pad3) -> /PWM3_Y-A
- J1 pad 4: unconnected-(J1-Pin_4-Pad4) -> GND
- J1 pad 5: unconnected-(J1-Pin_5-Pad5) -> +5V
- J1 pad 6: unconnected-(J1-Pin_6-Pad6) -> /AD1_U3
- J1 pad 7: unconnected-(J1-Pin_7-Pad7) -> /MOTOR3
- J1 pad 8: unconnected-(J1-Pin_8-Pad8) -> +3.3V
- J1 pad 9: unconnected-(J1-Pin_9-Pad9) -> GND
- J10 pad 1: unconnected-(J10-Pin_1-Pad1) -> /V_28V
- J10 pad 2: unconnected-(J10-Pin_2-Pad2) -> GND
- J10 pad 3: unconnected-(J10-Pin_3-Pad3) -> /MCU3_CAN2_L-
- J10 pad 4: unconnected-(J10-Pin_4-Pad4) -> /V_GND
- J10 pad 5: unconnected-(J10-Pin_5-Pad5) -> /MCU3_CAN2_H+
- J11 pad 1: unconnected-(J11-Pin_1-Pad1) -> /V_28V
- J11 pad 2: unconnected-(J11-Pin_2-Pad2) -> /V_GND
- J2 pad 1: unconnected-(J2-Pin_1-Pad1) -> +5V
- J2 pad 2: unconnected-(J2-Pin_2-Pad2) -> /PWM4_Z-B
- J2 pad 3: unconnected-(J2-Pin_3-Pad3) -> /PWM4_Y-A
- J2 pad 4: unconnected-(J2-Pin_4-Pad4) -> GND
- J2 pad 5: unconnected-(J2-Pin_5-Pad5) -> +5V
- J2 pad 6: unconnected-(J2-Pin_6-Pad6) -> /AD1_U4
- J2 pad 7: unconnected-(J2-Pin_7-Pad7) -> /MOTOR4
- J2 pad 8: unconnected-(J2-Pin_8-Pad8) -> +3.3V
- J2 pad 9: unconnected-(J2-Pin_9-Pad9) -> GND
- J3 pad 1: unconnected-(J3-Pin_1-Pad1) -> +5V
- J3 pad 2: unconnected-(J3-Pin_2-Pad2) -> /PWM7_Z-B
- J3 pad 3: unconnected-(J3-Pin_3-Pad3) -> /PWM7_Y-A
- J3 pad 4: unconnected-(J3-Pin_4-Pad4) -> GND
- J3 pad 5: unconnected-(J3-Pin_5-Pad5) -> +5V
- J3 pad 6: unconnected-(J3-Pin_6-Pad6) -> /AD1_U7
- J3 pad 7: unconnected-(J3-Pin_7-Pad7) -> /MOTOR7
- J3 pad 8: unconnected-(J3-Pin_8-Pad8) -> +3.3V
- J3 pad 9: unconnected-(J3-Pin_9-Pad9) -> GND
- J4 pad 1: unconnected-(J4-Pin_1-Pad1) -> +5V
- J4 pad 2: unconnected-(J4-Pin_2-Pad2) -> /PWM8_Z-B
- J4 pad 3: unconnected-(J4-Pin_3-Pad3) -> /PWM8_Y-A
- J4 pad 4: unconnected-(J4-Pin_4-Pad4) -> GND
- J4 pad 5: unconnected-(J4-Pin_5-Pad5) -> +5V
- J4 pad 6: unconnected-(J4-Pin_6-Pad6) -> /AD1_U8
- J4 pad 7: unconnected-(J4-Pin_7-Pad7) -> /MOTOR8
- J4 pad 8: unconnected-(J4-Pin_8-Pad8) -> +3.3V
- J4 pad 9: unconnected-(J4-Pin_9-Pad9) -> GND
- J5 pad 1: unconnected-(J5-Pin_1-Pad1) -> /V_28V
- J5 pad 2: unconnected-(J5-Pin_2-Pad2) -> /TX+
- J5 pad 3: unconnected-(J5-Pin_3-Pad3) -> /TX-
- J5 pad 4: unconnected-(J5-Pin_4-Pad4) -> /V_GND
- J5 pad 5: unconnected-(J5-Pin_5-Pad5) -> /RX-
- J5 pad 6: unconnected-(J5-Pin_6-Pad6) -> /RX+
- J5 pad 8: unconnected-(J5-Pin_8-Pad8) -> GND
- J8 pad 1: unconnected-(J8-Pin_1-Pad1) -> +5V
- J8 pad 2: unconnected-(J8-Pin_2-Pad2) -> GND
- J8 pad 3: unconnected-(J8-Pin_3-Pad3) -> /AD2_U3
- J8 pad 5: unconnected-(J8-Pin_5-Pad5) -> /AD2_U4
- J8 pad 6: unconnected-(J8-Pin_6-Pad6) -> GND
- J8 pad 7: unconnected-(J8-Pin_7-Pad7) -> +5V
- J9 pad 1: unconnected-(J9-Pin_1-Pad1) -> /V_28V
- J9 pad 2: unconnected-(J9-Pin_2-Pad2) -> GND
- J9 pad 3: unconnected-(J9-Pin_3-Pad3) -> /MCU2_CAN2_L-
- J9 pad 4: unconnected-(J9-Pin_4-Pad4) -> /V_GND
- J9 pad 5: unconnected-(J9-Pin_5-Pad5) -> /MCU2_CAN2_H+
Routing:
- net /TX+: track 0.00 -> 224.4 mm, vias 0 -> 1
- net /TX-: track 0.00 -> 215.5 mm, vias 0 -> 1
- net /RX+: track 0.00 -> 207.1 mm, vias 0 -> 1
- net /AD2_U3: track 0.00 -> 205.4 mm, vias 0 -> 1
- net /RX-: track 0.00 -> 203.3 mm, vias 0 -> 1
- net /AD2_U4: track 0.00 -> 197.2 mm, vias 0 -> 1
- net +5V: track 0.00 -> 128.1 mm
- net /MCU2_CAN2_L-: track 0.00 -> 109.8 mm, vias 0 -> 1
- net /MCU2_CAN2_H+: track 0.00 -> 104.4 mm, vias 0 -> 1
- net /AD1_U4: track 0.00 -> 68.0 mm, vias 0 -> 1
- net /MOTOR3: track 0.00 -> 62.1 mm, vias 0 -> 1
- net /AD1_U3: track 0.00 -> 58.1 mm, vias 0 -> 1
- net /MOTOR4: track 0.00 -> 57.8 mm
- net /PWM7_Y-A: track 0.00 -> 39.3 mm, vias 0 -> 1
- net /MCU3_CAN2_L-: track 0.00 -> 39.3 mm, vias 0 -> 1
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- added copper zone on B.Cu, net +3.3V
- added copper zone on In2.Cu, net +5V
- added copper zone on F.Cu, net /V_28V
- added copper zone on B.Cu, net /V_GND
- added copper zone on In2.Cu, net /V_GND
- added copper zone on B.Cu, net GND
- added copper zone on F.Cu, net GND
- added copper zone on In1.Cu, net GND
Other:
- outline, holes or cut-outs redrawn
- copper layers 2 -> 4
