File: EquipmentBox2/EquipmentBox2.kicad_pcb (KiCad board)
At the start: 2 copper layers, 272.5 x 41 mm, 11 parts, among them J1 UAC16-8, J10 UAC20-5, J11 UAC20-5, J2 UAC16-8, J3 UAC16-8, J4 UAC16-8, J5 UAC16-8, J6 UAC16-8, J7 UAC16-9, J8 UAC16-9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

Commit message: 已打样测试两版，第三版暂未修改
Parts:
- added J12: 430452412, Molex:430452412, B.Cu at (287.0, 59.5)
- added J13: 430452212, Molex:430452212, B.Cu at (316.0, 59.5)
- added J14: 430450612, Molex:430450612, B.Cu at (270.0, 59.5)
- added J15: UAC16-9, UACsocket:UAC16-9, F.Cu at (303.1, 46.5)
- added J16: XT60M, Connector_AMASS:AMASS_XT60-M_1x02_P7.20mm_Vertical, B.Cu at (185.6, 45.0)
- added J17: XT60F, Connector_AMASS:AMASS_XT60-F_1x02_P7.20mm_Vertical, B.Cu at (225.6, 45.0)
- added R1: 1K, Resistor_SMD:R_0402_1005Metric, F.Cu at (321.0, 44.0)
- added R2: 1K, Resistor_SMD:R_0402_1005Metric, F.Cu at (321.0, 47.0)
- added R3: 1K, Resistor_SMD:R_0402_1005Metric, F.Cu at (321.0, 50.0)
- added R4: 1K, Resistor_SMD:R_0402_1005Metric, F.Cu at (321.0, 53.0)
Connections:
- J1 pad 5: unconnected-(J1-Pin_5-Pad5) -> GND
- J1 pad 6: unconnected-(J1-Pin_6-Pad6) -> /CAN2_L-
- J1 pad 7: unconnected-(J1-Pin_7-Pad7) -> /CAN2_H+
- J11 pad 1: unconnected-(J11-Pin_1-Pad1) -> /V_28V
- J11 pad 2: unconnected-(J11-Pin_2-Pad2) -> GND
- J11 pad 3: unconnected-(J11-Pin_3-Pad3) -> /MCU1_CAN2_L-
- J11 pad 4: unconnected-(J11-Pin_4-Pad4) -> /V_GND
- J11 pad 5: unconnected-(J11-Pin_5-Pad5) -> /MCU1_CAN2_H+
- J4 pad 1: unconnected-(J4-Pin_1-Pad1) -> +12V
- J4 pad 4: unconnected-(J4-Pin_4-Pad4) -> GND
- J4 pad 6: unconnected-(J4-Pin_6-Pad6) -> /CAN1_L-
- J4 pad 7: unconnected-(J4-Pin_7-Pad7) -> /CAN1_H+
- J6 pad 1: unconnected-(J6-Pin_1-Pad1) -> +5V
- J6 pad 2: unconnected-(J6-Pin_2-Pad2) -> GND
- J6 pad 3: unconnected-(J6-Pin_3-Pad3) -> /AD2_U1
- J6 pad 5: unconnected-(J6-Pin_5-Pad5) -> /AD2_U2
- J6 pad 6: unconnected-(J6-Pin_6-Pad6) -> GND
- J6 pad 7: unconnected-(J6-Pin_7-Pad7) -> +5V
- J7 pad 1: unconnected-(J7-Pin_1-Pad1) -> +5V
- J7 pad 2: unconnected-(J7-Pin_2-Pad2) -> /PWM1_Z-B
- J7 pad 3: unconnected-(J7-Pin_3-Pad3) -> /PWM1_Y-A
- J7 pad 4: unconnected-(J7-Pin_4-Pad4) -> GND
- J7 pad 5: unconnected-(J7-Pin_5-Pad5) -> +5V
- J7 pad 6: unconnected-(J7-Pin_6-Pad6) -> /AD1_U1
- J7 pad 7: unconnected-(J7-Pin_7-Pad7) -> /MOTOR1
- J7 pad 8: unconnected-(J7-Pin_8-Pad8) -> +3.3V
- J7 pad 9: unconnected-(J7-Pin_9-Pad9) -> GND
- J8 pad 1: unconnected-(J8-Pin_1-Pad1) -> +5V
- J8 pad 2: unconnected-(J8-Pin_2-Pad2) -> /PWM2_Z-B
- J8 pad 3: unconnected-(J8-Pin_3-Pad3) -> /PWM2_Y-A
- J8 pad 4: unconnected-(J8-Pin_4-Pad4) -> GND
- J8 pad 5: unconnected-(J8-Pin_5-Pad5) -> +5V
- J8 pad 6: unconnected-(J8-Pin_6-Pad6) -> /AD1_U2
- J8 pad 7: unconnected-(J8-Pin_7-Pad7) -> /MOTOR2
- J8 pad 8: unconnected-(J8-Pin_8-Pad8) -> +3.3V
- J8 pad 9: unconnected-(J8-Pin_9-Pad9) -> GND
- J9 pad 1: unconnected-(J9-Pin_1-Pad1) -> +5V
- J9 pad 2: unconnected-(J9-Pin_2-Pad2) -> /PWM6_Z-B
- J9 pad 3: unconnected-(J9-Pin_3-Pad3) -> /PWM6_Y-A
- J9 pad 4: unconnected-(J9-Pin_4-Pad4) -> GND
- J9 pad 5: unconnected-(J9-Pin_5-Pad5) -> +5V
- J9 pad 6: unconnected-(J9-Pin_6-Pad6) -> /AD1_U6
- J9 pad 7: unconnected-(J9-Pin_7-Pad7) -> /MOTOR6
- J9 pad 8: unconnected-(J9-Pin_8-Pad8) -> +3.3V
- J9 pad 9: unconnected-(J9-Pin_9-Pad9) -> GND
Routing:
- net /CAN1_H+: track 0.00 -> 278.2 mm, vias 0 -> 1
- net /CAN1_L-: track 0.00 -> 274.7 mm, vias 0 -> 1
- net +12V: track 0.00 -> 271.5 mm
- net /CAN2_H+: track 0.00 -> 249.2 mm, vias 0 -> 1
- net /CAN2_L-: track 0.00 -> 246.1 mm, vias 0 -> 1
- net /AD2_U1: track 0.00 -> 209.9 mm, vias 0 -> 1
- net /AD2_U2: track 0.00 -> 201.7 mm, vias 0 -> 1
- net +5V: track 0.00 -> 128.1 mm
- net /AD1_U2: track 0.00 -> 68.0 mm, vias 0 -> 1
- net /MOTOR1: track 0.00 -> 62.1 mm, vias 0 -> 1
- net /AD1_U1: track 0.00 -> 58.1 mm, vias 0 -> 1
- net /MOTOR2: track 0.00 -> 57.8 mm
- net /PWM5_Y-A: track 0.00 -> 39.3 mm, vias 0 -> 1
- net /MCU1_CAN2_L-: track 0.00 -> 39.3 mm, vias 0 -> 1
- net /MOTOR5: track 0.00 -> 36.5 mm, vias 0 -> 1
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- added copper zone on B.Cu, net +3.3V
- added copper zone on In2.Cu, net +5V
- added copper zone on F.Cu, net /V_28V
- added copper zone on B.Cu, net /V_GND
- added copper zone on In2.Cu, net /V_GND
- added copper zone on B.Cu, net GND
- added copper zone on F.Cu, net GND
- added copper zone on In1.Cu, net GND
- added copper zone on In2.Cu, net GND
Other:
- outline, holes or cut-outs redrawn
- copper layers 2 -> 4
